File: PCB/Remote.kicad_pcb (KiCad board)
At the start: 2 copper layers, 192.4 x 50 mm, 136 parts, among them J1 USB_C_Receptacle_USB2.0, J2 Conn_01x50, J3 JST_PH_B2B-PH, J4 2.54x2 Header, Q1 DMG2301L, Q2 MBT3904DW1, Q3 DMG2301L, Q4 DMG2301L, Q5 DMG2301L, U1 MCP73831-2-OT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

Commit message: Removed font dependency
"Fredoka Light" font no longer needed
Parts:
- added kibuzzard-64A91BF0: G***, kibuzzard-64A91BF0, F.Cu at (92.8, 84.9)
- added kibuzzard-64A91C1C: G***, kibuzzard-64A91C1C, F.Cu at (92.8, 80.6)
- added kibuzzard-64A91C24: G***, kibuzzard-64A91C24, F.Cu at (95.4, 82.4)
Other:
- board text removed: "X"
- board text removed: "Y"
- board text removed: "Z"

Commit message: Added missing library components
Added the missing library symbols, footprints and 3D-models. These are all in a project-specific library called "omoteLib" (#19)
Parts:
- AE1: footprint mkern:RFANT5220110A2T -> omoteLib:RFANT5220110A2T
- D2: footprint mkern:LED_5mm_Side_Mount -> omoteLib:LED_5mm_Side_Mount
- J1: footprint mkern:USB_C_Receptacle_HRO_TYPE-C-31-M-12 -> omoteLib:USB_C_Receptacle_HRO_TYPE-C-31-M-12
- J2: footprint mkern:TFT_2.83IN_240X320_50PIN -> omoteLib:TFT_2.83IN_240X320_50PIN
- J3: footprint mkern:JST_PH_B2B-PH-SM4-TB_1x02-1MP_P2.00mm_Vertical -> omoteLib:JST_PH_B2B-PH-SM4-TB_1x02-1MP_P2.00mm_Vertical
- U5: footprint mkern:XDCR_LIS3DHTR -> omoteLib:XDCR_LIS3DHTR
- U6: footprint mkern:Heimdall vertical -> omoteLib:Heimdall vertical
- U7: footprint mkern:QFN-48-1EP_7x7mm_P0.5mm_EP5.3x5.3mm_ThermalVias_MR -> omoteLib:QFN-48-1EP_7x7mm_P0.5mm_EP5.3x5.3mm_ThermalVias_MR
Changed lines of the file:
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@@
       (stroke (width 0) (type solid)) (fill solid) (layer "F.SilkS"))
   )
-  (footprint "mkern:LED_5mm_Side_Mount" locked (layer "F.Cu")
+  (footprint "omoteLib:LED_5mm_Side_Mount" locked (layer "F.Cu")
     (at 59.676677 102 90)
     (descr "5mm LED for horizontal soldering to the board edge")
@@
     (pad "2" smd rect locked (at -1.275 3.5 90) (size 1.5 5) (layers "F.Cu" "F.Paste" "F.Mask")
       (net 14 "Net-(D2-A)") (pinfunction "A") (pintype "passive"))
-    (model "${KICAD_USER_3DMODEL_DIR}/Side Mount LED v1.step"
+    (model "${KIPRJMOD}/project_libraries/3D-models/Side Mount LED v1.step"
       (offset (xyz 0 0 0.25))
       (scale (xyz 1 1 1))
@@
     )
   )
-  (footprint "mkern:JST_PH_B2B-PH-SM4-TB_1x02-1MP_P2.00mm_Vertical" (layer "F.Cu")
+  (footprint "omoteLib:JST_PH_B2B-PH-SM4-TB_1x02-1MP_P2.00mm_Vertical" (layer "F.Cu")
     (at 224.9 113.5 90)
     (descr "JST PH series connector, B2B-PH-SM4-TB (http://www.jst-mfg.com/product/pdf/eng/ePH.pdf), generated with kicad-footprint-generator")
@@
     (pad "MP" smd roundrect (at -3.4 -1.75 90) (size 1.6 3) (layers "F.Cu" "F.Paste" "F.Mask") (roundrect_rratio 0.15625))
     (pad "MP" smd roundrect (at 3.4 -1.75 90) (size 1.6 3) (layers "F.Cu" "F.Paste" "F.Mask") (roundrect_rratio 0.15625))
-    (model "${KICAD_USER_3DMODEL_DIR}/B2B-PH-SM4-TB.STEP"
+    (model "${KIPRJMOD}/project_libraries/3D-models/B2B-PH-SM4-TB.STEP"
       (offset (xyz -4 3.25 0))
       (scale (xyz 1 1 1))
@@
     )
   )
-  (footprint "mkern:QFN-48-1EP_7x7mm_P0.5mm_EP5.3x5.3mm_ThermalVias_MR" (layer "F.Cu")
+  (footprint "omoteLib:QFN-48-1EP_7x7mm_P0.5mm_EP5.3x5.3mm_ThermalVias_MR" (layer "F.Cu")
     (at 76.85 91.55)
     (descr "QFN, 48 Pin (https://www.trinamic.com/fileadmin/assets/Products/ICs_Documents/TMC2041_datasheet.pdf#page=62), generated with kicad-footprint-generator ipc_noLead_generator.py")
@@
     )
   )
-  (footprint "mkern:XDCR_LIS3DHTR" (layer "F.Cu")
+  (footprint "omoteLib:XDCR_LIS3DHTR" (layer "F.Cu")
     (at 89.75 84.786992 90)
     (property "MANUFACTURER" "STMicroelectronics")
@@
     (pad "16" smd rect (at -0.5 -1.3 180) (size 0.8 0.3) (layers "F.Cu" "F.Paste" "F.Mask")
       (net 98 "unconnected-(U5-ADC1-Pad16)") (pinfunction "ADC1") (pintype "input+no_connect") (solder_paste_margin_ratio -0.05))
-    (model "${KICAD_USER_3DMODEL_DIR}/LIS3DHTR.step"
+    (model "${KIPRJMOD}/project_libraries/3D-models/LIS3DHTR.step"
       (offset (xyz 0 0 0))
       (scale (xyz 1 1 1))
@@
       (stroke (width 0) (type solid)) (fill solid) (layer "F.Mask"))
   )
-  (footprint "mkern:TFT_2.83IN_240X320_50PIN" locked (layer "F.Cu")
+  (footprint "omoteLib:TFT_2.83IN_240X320_50PIN" locked (layer "F.Cu")
     (at 91.622852 102 90)
     (property "Sheetfile" "Remote.kicad_sch")
@@
     (pad "MP" smd roundrect locked (at 14.35 13.09 270) (size 2.4 2.4) (layers "F.Cu" "F.Paste" "F.Mask") (roundrect_rratio 0.125)
       (net 48 "GND") (pinfunction "MP") (pintype "passive") (solder_mask_margin 0.1016))
-    (model "${KICAD_USER_3DMODEL_DIR}/541325062_colored.step"
+    (model "${KIPRJMOD}/project_libraries/3D-models/541325062_colored.step"
       (offset (xyz 0 -15.5 0))
       (scale (xyz 1 1 1))
       (rotate (xyz 0 0 0))
     )
-    (model "${KICAD_USER_3DMODEL_DIR}/280QV10 v5.step"
+    (model "${KIPRJMOD}/project_libraries/3D-models/280QV10 v5.step"
       (offset (xyz 0 -22.25 -6))
       (scale (xyz 1 1 1))
@@
     )
   )
-  (footprint "mkern:Heimdall vertical" (layer "F.Cu")
+  (footprint "omoteLib:Heimdall vertical" (layer "F.Cu")
     (at 55.4 116.3 90)
     (descr "VISHAY Heimdall for TSSP77038")
@@
     (pad "4" smd rect (at 1.9 0.7 180) (size 2 0.8) (layers "F.Cu" "F.Paste" "F.Mask")
       (net 48 "GND") (pinfunction "GND") (pintype "power_in"))
-    (model "${KICAD_USER_3DMODEL_DIR}/82672Heimdall.stp"
+    (model "${KIPRJMOD}/project_libraries/3D-models/82672Heimdall.stp"
       (offset (xyz 0 -1.2 1.6))
       (scale (xyz 1 1 1))
@@
     )
   )
-  (footprint "mkern:RFANT5220110A2T" (layer "F.Cu")
+  (footprint "omoteLib:RFANT5220110A2T" (layer "F.Cu")
     (at 55.500146 85.711992)
     (descr "Walsin RFANT5220110A2T SMD antenna 2400-2500Mhz, 2dBi, http://www.passivecomponent.com/wp-content/uploads/2013/12/ASC_RFANT5220110A2T_V03.pdf")
@@
     (pad "1" smd roundrect (at 2.7 0 180) (size 1 2) (layers "F.Cu" "F.Paste" "F.Mask") (roundrect_rratio 0.208333)
       (net 3 "Net-(AE1-A)") (pinfunction "A") (pintype "input"))
-    (model "${KICAD_USER_3DMODEL_DIR}/Walsin RFANT5220110A2T v1.step"
+    (model "${KIPRJMOD}/project_libraries/3D-models/Walsin RFANT5220110A2T v1.step"
       (offset (xyz 0 0 0))
       (scale (xyz 1 1 1))
@@
     )
   )
-  (footprint "mkern:USB_C_Receptacle_HRO_TYPE-C-31-M-12" (layer "F.Cu")
+  (footprint "omoteLib:USB_C_Receptacle_HRO_TYPE-C-31-M-12" (layer "F.Cu")
     (at 241 102 90)
     (descr "USB Type-C receptacle for USB 2.0 and PD, http://www.krhro.com/uploads/soft/180320/1-1P320120243.pdf")
