File: PCB/Remote.kicad_sch (KiCad schematic)
At the start: 121 parts, among them J1 USB_C_Receptacle_USB2.0, J2 Conn_01x50, J3 JST_PH_B2B-PH, J4 2.54x2 Header, Q1 DMG2301L, Q2 MBT3904DW1, Q3 DMG2301L, Q4 DMG2301L, Q5 DMG2301L, U1 MCP73831-2-OT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

Commit message: Added missing library components
Added the missing library symbols, footprints and 3D-models. These are all in a project-specific library called "omoteLib" (#19)
Parts:
- AE1: footprint mkern:RFANT5220110A2T -> omoteLib:RFANT5220110A2T
- D2: footprint mkern:LED_5mm_Side_Mount -> omoteLib:LED_5mm_Side_Mount
- J1: footprint mkern:USB_C_Receptacle_HRO_TYPE-C-31-M-12 -> omoteLib:USB_C_Receptacle_HRO_TYPE-C-31-M-12
- J2: footprint mkern:TFT_2.83IN_240X320_50PIN -> omoteLib:TFT_2.83IN_240X320_50PIN; symbol mkern:Conn_01x50 -> omoteLib:Conn_01x50
- J3: footprint mkern:JST_PH_B2B-PH-SM4-TB_1x02-1MP_P2.00mm_Vertical -> omoteLib:JST_PH_B2B-PH-SM4-TB_1x02-1MP_P2.00mm_Vertical
- U4: symbol mkern:USBLC6-2P6 -> omoteLib:USBLC6-2P6
- U5: symbol mkern:LIS3DHTR -> omoteLib:LIS3DHTR
- U6: footprint mkern:Heimdall vertical -> omoteLib:Heimdall vertical
- U7: footprint mkern:QFN-48-1EP_7x7mm_P0.5mm_EP5.3x5.3mm_ThermalVias_MR -> omoteLib:QFN-48-1EP_7x7mm_P0.5mm_EP5.3x5.3mm_ThermalVias_MR
Changed lines of the file:
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@@
       (effects (font (size 1.27 1.27)))
     )
-    (property "Footprint" "mkern:Heimdall vertical" (at 256.54 213.36 0)
+    (property "Footprint" "omoteLib:Heimdall vertical" (at 256.54 213.36 0)
       (effects (font (size 1.27 1.27)) hide)
     )
@@
     )
   )
-  (symbol (lib_id "mkern:LIS3DHTR") (at 360.68 49.53 0) (mirror y) (unit 1)
+  (symbol (lib_id "omoteLib:LIS3DHTR") (at 360.68 49.53 0) (mirror y) (unit 1)
     (in_bom yes) (on_board yes) (dnp no) (fields_autoplaced)
     (property "Reference" "U5" (at 360.68 30.48 0)
@@
       (effects (font (size 1.27 1.27)))
     )
-    (property "Footprint" "mkern:USB_C_Receptacle_HRO_TYPE-C-31-M-12" (at 39.37 50.8 0)
+    (property "Footprint" "omoteLib:USB_C_Receptacle_HRO_TYPE-C-31-M-12" (at 39.37 50.8 0)
       (effects (font (size 1.27 1.27)) hide)
     )
@@
       (effects (font (size 1.27 1.27)) (justify right))
     )
-    (property "Footprint" "mkern:JST_PH_B2B-PH-SM4-TB_1x02-1MP_P2.00mm_Vertical" (at 116.84 170.18 0)
+    (property "Footprint" "omoteLib:JST_PH_B2B-PH-SM4-TB_1x02-1MP_P2.00mm_Vertical" (at 116.84 170.18 0)
       (effects (font (size 1.27 1.27)) hide)
     )
@@
     )
   )
-  (symbol (lib_id "mkern:USBLC6-2P6") (at 78.74 46.99 0) (unit 1)
+  (symbol (lib_id "omoteLib:USBLC6-2P6") (at 78.74 46.99 0) (unit 1)
     (in_bom yes) (on_board yes) (dnp no)
     (property "Reference" "U4" (at 71.12 38.1 0)
@@
       (effects (font (size 1.27 1.27)) (justify right))
     )
-    (property "Footprint" "mkern:LED_5mm_Side_Mount" (at 200.025 217.17 0)
+    (property "Footprint" "omoteLib:LED_5mm_Side_Mount" (at 200.025 217.17 0)
       (effects (font (size 1.27 1.27)) hide)
     )
@@
     )
   )
-  (symbol (lib_id "mkern:Conn_01x50") (at 384.81 172.72 0) (unit 1)
+  (symbol (lib_id "omoteLib:Conn_01x50") (at 384.81 172.72 0) (unit 1)
     (in_bom yes) (on_board yes) (dnp no)
     (property "Reference" "J2" (at 378.46 105.41 0)
@@
       (effects (font (size 1.27 1.27)) (justify left))
     )
-    (property "Footprint" "mkern:TFT_2.83IN_240X320_50PIN" (at 386.08 241.3 0)
+    (property "Footprint" "omoteLib:TFT_2.83IN_240X320_50PIN" (at 386.08 241.3 0)
       (effects (font (size 1.27 1.27)) hide)
     )
@@
       (effects (font (size 1.27 1.27)) (justify left))
     )
-    (property "Footprint" "mkern:QFN-48-1EP_7x7mm_P0.5mm_EP5.3x5.3mm_ThermalVias_MR" (at 238.76 119.38 0)
+    (property "Footprint" "omoteLib:QFN-48-1EP_7x7mm_P0.5mm_EP5.3x5.3mm_ThermalVias_MR" (at 238.76 119.38 0)
       (effects (font (size 1.27 1.27)) hide)
     )
@@
       (effects (font (size 1.27 1.27)) (justify left))
     )
-    (property "Footprint" "mkern:RFANT5220110A2T" (at 285.75 24.13 0)
-      (effects (font (size 1.27 1.27)) hide)
-    )
+    (property "Footprint" "omoteLib:RFANT5220110A2T" (at 285.75 24.13 0)
+      (effects (font (size 1.27 1.27)) hide)
+    )
