File: PCB/Revision 4 (deprecated)/Omote.kicad_sch (KiCad schematic)
At the start: 172 parts, among them J1 USB_C_Receptacle_USB2.0, J2 Conn_01x50, J3 JST_PH_B2B-PH, J4 2.54x2 Header, J5 Micro_SD_Card, Q1 DMG2301L, Q2 MBT3904DW1, Q3 DMG2301L, Q4 DMG2301L, Q5 DMG2301L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

Commit message: REV5 hardware added
TODO: update production files and BOMs
Parts:
- removed C29: 100nF, Capacitor_SMD:C_0603_1608Metric, symbol Device:C
- removed D10, D11, D12, D13, D14, D15, D16, D6, D7, D8, D9: LED, LED_SMD:LED_0603_1608Metric, symbol Device:LED
- removed J5: Micro_SD_Card, omoteLib:MicroSD Slot TF-01A, symbol Connector:Micro_SD_Card_Det1
- removed Q7: DMG2301L, Package_TO_SOT_SMD:SOT-23, symbol Transistor_FET:DMG2301L
- removed R10, R24: 10k, Resistor_SMD:R_0603_1608Metric, symbol Device:R
- removed R2: 330, Resistor_SMD:R_0603_1608Metric, symbol Device:R
- removed R38, R41, R42, R43, R44: 2k2, Resistor_SMD:R_0603_1608Metric, symbol Device:R
- removed TP14, TP15, TP16, TP17, TP18, TP19, TP20, TP21, TP22, TP23: TestPoint, TestPoint:TestPoint_Pad_D1.5mm, symbol Connector:TestPoint
- removed U12: TCA8418, Package_DFN_QFN:HVQFN-24-1EP_4x4mm_P0.5mm_EP2.5x2.5mm, symbol omoteLib:TCA8418
- removed U7: ESP32-S3-WROOM-1-N16R8, RF_Module:ESP32-S3-WROOM-1, symbol RF_Module:ESP32-S3-WROOM-1
- added AE1: Antenna, omoteLib:RFANT5220110A2T, symbol Device:Antenna
- added C19: 1.2pF, Capacitor_SMD:C_0603_1608Metric, symbol Device:C
- added U7: ESP32-PICO-D4, omoteLib:QFN-48-1EP_7x7mm_P0.5mm_EP5.3x5.3mm_ThermalVias_MR, symbol RF_Module:ESP32-PICO-D4
- C11: value 10uF -> 2.2uF; footprint Capacitor_SMD:C_0805_2012Metric -> Capacitor_SMD:C_0603_1608Metric; LCSC C15850 -> C913904
- C14: value 10uF -> 100nF; footprint Capacitor_SMD:C_0805_2012Metric -> Capacitor_SMD:C_0603_1608Metric; LCSC C15850 -> C1591
- C18: value 10uF -> 1.2pF; footprint Capacitor_SMD:C_0805_2012Metric -> Capacitor_SMD:C_0603_1608Metric; LCSC C15850 -> (none); now not fitted; now left out of the parts list
- D1: value BAT20J -> MBR0520; footprint Diode_SMD:D_SOD-323 -> Diode_SMD:D_SOD-123; LCSC C155590 -> C475717
- D2: value SFH4547 -> SFH4547
- H4: footprint MountingHole:MountingHole_3.2mm_M3 -> MountingHole:MountingHole_3.2mm_M3_Pad_Via
- R23, R31, R32, R33, R34, R35: value 2k2 -> 10k; LCSC C114662 -> C98220
- R36: value 10k -> 0; LCSC C98220 -> C116699
- U6: LCSC C3291489 -> C499566
Connections:
- net LCD_D0 is gone; now on net GND: J2.32 (Pin_32)
- net LCD_D1 is gone; now on net GND: J2.31 (Pin_31)
- net LCD_D2 is gone; now on net GND: J2.30 (Pin_30)
- net LCD_D3 is gone; now on net GND: J2.29 (Pin_29)
- net LCD_D4 is gone; now on net GND: J2.28 (Pin_28)
- net LCD_D5 is gone; now on net GND: J2.27 (Pin_27)
- net LCD_D6 is gone; now on net GND: J2.26 (Pin_26)
- net LCD_D7 is gone; now on net GND: J2.25 (Pin_25)
- net LCD_WR is gone; now on net LCD_DC: J2.36 (Pin_36)
- net SW_BL is gone; now on net GND: C14.2
- net SW_PWR is gone; now on net SW_D: S17.2
- net +3.3V: now also C11.1, C14.1, R23.2, U7.1 (VDDA), U7.19 (VDD3P3_RTC), U7.3 (VDDA3P3), U7.37 (VDD3P3_CPU), U7.4 (VDDA3P3), U7.43 (VDDA), U7.46 (VDDA); no longer C11.2, R36.2
- net +VSW: now also J2.7 (Pin_7), J2.8 (Pin_8), J2.9 (Pin_9)
- net ACC_INT: now also U7.20 (IO13)
- net CRG_STAT: now also R23.1, U7.42 (IO21)
- net ESP_EN: now also U7.9 (EN)
- net GND: now also C11.2, J2.11 (Pin_11), J2.12 (Pin_12), J2.13 (Pin_13), J2.14 (Pin_14), R31.2, R32.2, R33.2, R34.2, R35.2, C19.1, U7.49 (GND); no longer C11.1, C14.1, J2.7 (Pin_7), J2.8 (Pin_8), J2.9 (Pin_9), R23.1, R31.1, R32.1, R33.1, R34.1, R35.1, S17.1
- net IO0: now also U7.23 (IO0)
- net IR_LED: now also U7.13 (IO33)
- net IR_RX: now also U7.21 (IO15)
- net IR_VCC: now also U7.14 (IO25)
- net LCD_BL: now also U7.24 (IO4)
- net LCD_CS: now also U7.34 (IO5)
- net LCD_DC: now also U7.28 (SD2/IO9); no longer J2.37 (Pin_37)
- net LCD_EN: now also U7.29 (SD3/IO10)
- net SCL: now also U7.39 (IO22)
- net SDA: now also U7.38 (IO19)
- net SW_1: now also U7.12 (IO32)
- net SW_2: now also S17.1, U7.15 (IO26)
- net SW_3: now also U7.16 (IO27)
- net SW_4: now also U7.17 (IO14)
- net SW_5: now also U7.18 (IO12)
- net SW_A: now also R31.1, U7.6 (SENSOR_CAPP)
- net SW_B: now also R32.1, U7.7 (SENSOR_CAPN)
- net SW_C: now also R33.1, U7.8 (SENSOR_VN)
- net SW_D: now also R34.1, U7.10 (IO34)
- net SW_E: now also R35.1, U7.11 (IO35)
- net USB_RXD: now also U7.40 (U0RXD/IO3)
- net USB_TXD: now also U7.41 (U0TXD/IO1)
- net at D3.2 (A): now also U7.22 (IO2)
- net LCD_MOSI: now reaches J2.34 (Pin_34)
- net LCD_MOSI: now also U7.36 (IO23)
- net LCD_RD: no longer names the net of J2.35 (Pin_35)
- net SD_3V3: no longer names the net of C18.2
- net SD_3V3: now also R36.2, U7.2 (LNA_IN)
- net TCA_INT: no longer names the net of R36.1
- net TCA_INT: now also AE1.1 (A), C19.2
- net USB_3V3: no longer names the net of C24.1, C4.1, U3.16 (VCC), U3.4 (V3), U8.5 (VOUT)
- new net LCD_SCK: J2.37 (Pin_37), U7.35 (IO18)
- no-connect marks 28 -> 25
Other:
- note added: "Boot Mode Configuration: Pin Default Boot Download GPIO0 1 1 0 U0TXD 1 1 x GPIO2 0 x 0 GPIO4 0 x x MTDO 1 x x GPIO5 1 1 x If U0TXD, GPIO2, GPIO5 are floating, GPIO0 determines boot mode"
- note added: "Button Matrix"
- note added: "Charge current: R_PROG = 4.7k IBAT = ca. 280mA"
- note added: "Pull-Down resistors needed for ext1 interrupt"
- note added: "RTC GPIO: 0,2,4,12-15,25-27,32-39 ext0: - single RTC_GPIO as wakeup source ext1: - multiple RTC_GPIOs as wakeup source - either any pin high or all pins low - internal Pull-ups /Pull-downs disabled"
- note removed: "Alternative Part: Everlight Elec IRM-V838M3-C/TR1"
- note removed: "Button Matrix and GPIO Expander"
- note removed: "Charge current: R_PROG = 4.7k IBAT = ca. 213mA"
- note removed: "Keyboard Backlight"
- note removed: "Keyboard Matrix I2C address: 0x34"
- note removed: "Power off microSD in sleep mode"
- note removed: "RTC GPIO: 1-20 Bootstraps: 0,3,45,46 ext0: - single RTC_GPIO as wakeup source ext1: - multiple RTC_GPIOs as wakeup source - either any pin high or any pin low - internal Pull-ups /Pull-downs disabled"
- note removed: "µSD Connector"
- moved on the sheet: C1, C12, C13, C15, C16, C20, C21, C22, C23, C25, C26, C27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
